File: CH340-USB-C/CH340-USB-C.kicad_sch (KiCad schematic)
At the start: 24 parts, among them J1 USB_C_Receptacle_USB2.0, J2 Conn_01x05_Female, SW1 SW_Push_SPDT, U1 XC6206PxxxMR, U2 CH340N

Commit message: 新佈局&USB 信號
Parts:
- TP1, TP2, TP3, TP4, TP5, TP6: footprint TestPoint:TestPoint_Pad_D2.0mm -> TestPoint:TestPoint_Pad_D1.0mm; now left out of the parts list
Changed lines of the file:
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@@
   )
   (symbol (lib_id "Connector:TestPoint") (at 207.01 73.025 90) (unit 1)
-    (in_bom yes) (on_board yes) (fields_autoplaced)
+    (in_bom no) (on_board yes) (fields_autoplaced)
     (property "Reference" "TP5" (id 0) (at 203.708 66.675 90))
     (property "Value" "TestPoint" (id 1) (at 203.708 69.215 90))
-    (property "Footprint" "TestPoint:TestPoint_Pad_D2.0mm" (id 2) (at 207.01 67.945 0)
+    (property "Footprint" "TestPoint:TestPoint_Pad_D1.0mm" (id 2) (at 207.01 67.945 0)
       (effects (font (size 1.27 1.27)) hide)
     )
@@
   )
   (symbol (lib_id "Connector:TestPoint") (at 207.01 38.1 90) (unit 1)
-    (in_bom yes) (on_board yes) (fields_autoplaced)
+    (in_bom no) (on_board yes) (fields_autoplaced)
     (property "Reference" "TP1" (id 0) (at 203.708 31.75 90))
     (property "Value" "TestPoint" (id 1) (at 203.708 34.29 90))
-    (property "Footprint" "TestPoint:TestPoint_Pad_D2.0mm" (id 2) (at 207.01 33.02 0)
+    (property "Footprint" "TestPoint:TestPoint_Pad_D1.0mm" (id 2) (at 207.01 33.02 0)
       (effects (font (size 1.27 1.27)) hide)
     )
@@
   )
   (symbol (lib_id "Connector:TestPoint") (at 207.01 46.99 90) (unit 1)
-    (in_bom yes) (on_board yes) (fields_autoplaced)
+    (in_bom no) (on_board yes) (fields_autoplaced)
     (property "Reference" "TP2" (id 0) (at 203.708 40.64 90))
     (property "Value" "TestPoint" (id 1) (at 203.708 43.18 90))
-    (property "Footprint" "TestPoint:TestPoint_Pad_D2.0mm" (id 2) (at 207.01 41.91 0)
+    (property "Footprint" "TestPoint:TestPoint_Pad_D1.0mm" (id 2) (at 207.01 41.91 0)
       (effects (font (size 1.27 1.27)) hide)
     )
@@
   )
   (symbol (lib_id "Connector:TestPoint") (at 207.01 64.77 90) (unit 1)
-    (in_bom yes) (on_board yes) (fields_autoplaced)
+    (in_bom no) (on_board yes) (fields_autoplaced)
     (property "Reference" "TP4" (id 0) (at 203.708 58.42 90))
     (property "Value" "TestPoint" (id 1) (at 203.708 60.96 90))
-    (property "Footprint" "TestPoint:TestPoint_Pad_D2.0mm" (id 2) (at 207.01 59.69 0)
+    (property "Footprint" "TestPoint:TestPoint_Pad_D1.0mm" (id 2) (at 207.01 59.69 0)
       (effects (font (size 1.27 1.27)) hide)
     )
@@
   )
   (symbol (lib_id "Connector:TestPoint") (at 207.01 55.88 90) (unit 1)
-    (in_bom yes) (on_board yes) (fields_autoplaced)
+    (in_bom no) (on_board yes) (fields_autoplaced)
     (property "Reference" "TP3" (id 0) (at 203.708 49.53 90))
     (property "Value" "TestPoint" (id 1) (at 203.708 52.07 90))
-    (property "Footprint" "TestPoint:TestPoint_Pad_D2.0mm" (id 2) (at 207.01 50.8 0)
+    (property "Footprint" "TestPoint:TestPoint_Pad_D1.0mm" (id 2) (at 207.01 50.8 0)
       (effects (font (size 1.27 1.27)) hide)
     )
@@
   )
   (symbol (lib_id "Connector:TestPoint") (at 207.01 81.28 90) (unit 1)
-    (in_bom yes) (on_board yes) (fields_autoplaced)
+    (in_bom no) (on_board yes) (fields_autoplaced)
     (property "Reference" "TP6" (id 0) (at 203.708 74.93 90))
     (property "Value" "TestPoint" (id 1) (at 203.708 77.47 90))
-    (property "Footprint" "TestPoint:TestPoint_Pad_D2.0mm" (id 2) (at 207.01 76.2 0)
+    (property "Footprint" "TestPoint:TestPoint_Pad_D1.0mm" (id 2) (at 207.01 76.2 0)
       (effects (font (size 1.27 1.27)) hide)
     )
@@
     )
     (path "/92b3f96e-4673-4f7c-84d5-9cc858573923"
-      (reference "TP1") (unit 1) (value "TestPoint") (footprint "TestPoint:TestPoint_Pad_D2.0mm")
+      (reference "TP1") (unit 1) (value "TestPoint") (footprint "TestPoint:TestPoint_Pad_D1.0mm")
     )
     (path "/96066fe1-f77b-478d-9b2d-0f1adc727f12"
-      (reference "TP2") (unit 1) (value "TestPoint") (footprint "TestPoint:TestPoint_Pad_D2.0mm")
+      (reference "TP2") (unit 1) (value "TestPoint") (footprint "TestPoint:TestPoint_Pad_D1.0mm")
     )
     (path "/d9461d13-f8bc-497b-b540-f733f84103d7"
-      (reference "TP3") (unit 1) (value "TestPoint") (footprint "TestPoint:TestPoint_Pad_D2.0mm")
+      (reference "TP3") (unit 1) (value "TestPoint") (footprint "TestPoint:TestPoint_Pad_D1.0mm")
     )
     (path "/98476643-1dc3-4cb2-875f-ffa29d752e72"
-      (reference "TP4") (unit 1) (value "TestPoint") (footprint "TestPoint:TestPoint_Pad_D2.0mm")
+      (reference "TP4") (unit 1) (value "TestPoint") (footprint "TestPoint:TestPoint_Pad_D1.0mm")
     )
     (path "/1ed8b24b-cd25-4583-98e4-aed9a7451e4a"
-      (reference "TP5") (unit 1) (value "TestPoint") (footprint "TestPoint:TestPoint_Pad_D2.0mm")
+      (reference "TP5") (unit 1) (value "TestPoint") (footprint "TestPoint:TestPoint_Pad_D1.0mm")
     )
     (path "/fbf8ac89-c320-46e2-b575-18008179d8e3"
-      (reference "TP6") (unit 1) (value "TestPoint") (footprint "TestPoint:TestPoint_Pad_D2.0mm")
+      (reference "TP6") (unit 1) (value "TestPoint") (footprint "TestPoint:TestPoint_Pad_D1.0mm")
     )
     (path "/588c1e41-6e7d-4663-9833-3ee3d386ce28"

Commit message: 更新佈局
Connections:
- net +3V3: now also SW1.1 (A); no longer SW1.3 (C)
- net +5V: now also SW1.3 (C); no longer SW1.1 (A)
Changed lines of the file:
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@@
     (stroke (width 0) (type solid) (color 0 0 0 0))
   )
-  (wire (pts (xy 134.62 122.555) (xy 146.685 122.555))
+  (wire (pts (xy 146.685 115.57) (xy 146.685 117.475))
     (stroke (width 0) (type default) (color 0 0 0 0))
   )
@@
     (stroke (width 0) (type solid) (color 0 0 0 0))
   )
-  (wire (pts (xy 134.62 117.475) (xy 140.97 117.475))
-    (stroke (width 0) (type default) (color 0 0 0 0))
-  )
   (wire (pts (xy 47.625 33.02) (xy 65.405 33.02))
     (stroke (width 0) (type solid) (color 0 0 0 0))
@@
     (stroke (width 0) (type default) (color 0 0 0 0))
   )
+  (wire (pts (xy 146.685 117.475) (xy 134.62 117.475))
+    (stroke (width 0) (type default) (color 0 0 0 0))
+  )
   (wire (pts (xy 207.01 46.99) (xy 218.44 46.99))
     (stroke (width 0) (type default) (color 0 0 0 0))
@@
   )
   (wire (pts (xy 207.01 64.77) (xy 218.44 64.77))
+    (stroke (width 0) (type default) (color 0 0 0 0))
+  )
+  (wire (pts (xy 134.62 122.555) (xy 152.4 122.555))
     (stroke (width 0) (type default) (color 0 0 0 0))
   )
@@
     (pin "1")
   )
-  (symbol (lib_id "power:+5V") (at 140.97 117.475 0) (unit 1)
-    (in_bom yes) (on_board yes) (fields_autoplaced)
-    (property "Reference" "#PWR015" (id 0) (at 140.97 121.285 0)
-      (effects (font (size 1.27 1.27)) hide)
-    )
-    (property "Value" "+5V" (id 1) (at 140.97 112.395 0))
-    (property "Footprint" "" (id 2) (at 140.97 117.475 0)
-      (effects (font (size 1.27 1.27)) hide)
-    )
-    (property "Datasheet" "" (id 3) (at 140.97 117.475 0)
+  (symbol (lib_id "power:+5V") (at 152.4 122.555 0) (unit 1)
+    (in_bom yes) (on_board yes) (fields_autoplaced)
+    (property "Reference" "#PWR015" (id 0) (at 152.4 126.365 0)
+      (effects (font (size 1.27 1.27)) hide)
+    )
+    (property "Value" "+5V" (id 1) (at 152.4 117.475 0))
+    (property "Footprint" "" (id 2) (at 152.4 122.555 0)
+      (effects (font (size 1.27 1.27)) hide)
+    )
+    (property "Datasheet" "" (id 3) (at 152.4 122.555 0)
       (effects (font (size 1.27 1.27)) hide)
     )
@@
     (pin "1")
   )
-  (symbol (lib_id "power:+3V3") (at 146.685 122.555 0) (unit 1)
-    (in_bom yes) (on_board yes) (fields_autoplaced)
-    (property "Reference" "#PWR016" (id 0) (at 146.685 126.365 0)
-      (effects (font (size 1.27 1.27)) hide)
-    )
-    (property "Value" "+3V3" (id 1) (at 146.685 117.475 0))
-    (property "Footprint" "" (id 2) (at 146.685 122.555 0)
-      (effects (font (size 1.27 1.27)) hide)
-    )
-    (property "Datasheet" "" (id 3) (at 146.685 122.555 0)
-      (effects (font (size 1.27 1.27)) hide)
-    )
+  (symbol (lib_id "power:+3V3") (at 146.685 115.57 0) (unit 1)
+    (in_bom yes) (on_board yes) (fields_autoplaced)
+    (property "Reference" "#PWR016" (id 0) (at 146.685 119.38 0)
+      (effects (font (size 1.27 1.27)) hide)
+    )
+    (property "Value" "+3V3" (id 1) (at 146.685 110.49 0))
+    (property "Footprint" "" (id 2) (at 146.685 115.57 0)
+      (effects (font (size 1.27 1.27)) hide)
+    )
+    (property "Datasheet" "" (id 3) (at 146.685 115.57 0)
+      (effects (font (size 1.27 1.27)) hide)
+    )

Commit message: 鋪銅絲印
Parts:
- removed TP1, TP2, TP3, TP4, TP5, TP6: TestPoint, TestPoint:TestPoint_Pad_D1.0mm, symbol Connector:TestPoint

Commit message: 將排真座排除BOM
Parts:
- J2: now left out of the parts list
Changed lines of the file:
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@@
   )
   (symbol (lib_id "Connector:Conn_01x05_Female") (at 128.27 165.735 180) (unit 1)
-    (in_bom yes) (on_board yes) (fields_autoplaced)
+    (in_bom no) (on_board yes) (fields_autoplaced)
     (property "Reference" "J2" (id 0) (at 127 167.0051 0)
       (effects (font (size 1.27 1.27)) (justify left))
