File: CH340-USB-C/CH340-USB-C.kicad_pcb (KiCad board)
At the start: 2 copper layers, 37.2 x 17.8 mm, 20 parts, among them J1 USB_C_Receptacle_USB2.0, J2 Conn_01x04_MountingPin, SW1 SW_Push_SPDT, U1 XC6206PxxxMR, U2 CH340N

Commit message: 增加絲印
增加公司名稱及腳位名稱
Parts:
- moved REF** 18.7 mm to (78.9, 102.9), turned to 180 degrees
Other:
- board text added: "GND"
- board text added: "仲宇電氣"

Commit message: 打樣
Parts:
- moved REF** 18.7 mm to (96.6, 97.0), turned to -90 degrees
Other:
- board text removed: "GND"
- board text removed: "仲宇電氣"
